File: pressure-sensor-pcb/pressure-sensor-pcb.kicad_sch (KiCad schematic)
At the start: 2 parts

Commit message: add footprints
Parts:
- J?: footprint (none) -> Connector_PinHeader_2.54mm:PinHeader_2x24_P2.54mm_Vertical

Commit message: test initial PCB layout for fit
Parts:
- XA1: renamed from XA?; footprint Arduino_Library:Arduino_Uno_Shield -> Arduino:Arduino_Uno_Shield
- gave numbers to parts that had none: 1
